File: esp32.kicad_sch (KiCad schematic)
At the start: 4 parts, among them J3 Conn_01x05, J4 Conn_01x10, J5 Conn_01x05, U5 ESP32-C3-MINI-1-N4

Commit message: 2022-06-20
Connections:
- net Earth: now also U5.53 (GND)
Changed lines of the file:
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@@
     (pin "51")
     (pin "52")
+    (pin "53")
     (pin "6")
     (pin "7")
