File: fishbite.kicad_pcb (KiCad board)
At the start: 2 copper layers, 43 parts, among them IC1 ADXL345BCCZ-RL, J1 Batt, U1 USB4130-GF-C, U2 MCP73831-2-OT, U3 CC2640R2FRHBR, U4 MIC5317-3.3YM5-TR, Y1 32.768kHz, Y2 24MHz

Commit message: 2022-06-14
Parts:
- added D1: RG_LED, APBA3010SURKCGKC-GX:APBA3010SURKCGKC-GX, F.Cu at (180.6, 70.8)
- added J2: test, Connector_PinHeader_2.54mm:PinHeader_2x14_P2.54mm_Vertical, F.Cu at (179.9, 33.4)
- added R2: 10k/1608, Resistor_SMD:R_0603_1608Metric_Pad0.98x0.95mm_HandSolder, F.Cu at (179.8, 73.7)
- added R3: 10k/1608, Resistor_SMD:R_0603_1608Metric_Pad0.98x0.95mm_HandSolder, F.Cu at (191.3, 32.3)
- added R4: 100/1608, Resistor_SMD:R_0603_1608Metric_Pad0.98x0.95mm_HandSolder, F.Cu at (187.0, 32.3)
- moved C20 135.6 mm to (51.0, 107.0), turned to 180 degrees
- moved C18 130.7 mm to (44.0, 95.5)
- moved Y1 124.7 mm to (46.0, 93.8)
- moved C13 122.3 mm to (51.5, 83.5), turned to 180 degrees
- moved R1 120.0 mm to (51.0, 108.5), turned to 180 degrees
- moved C12 119.5 mm to (50.0, 88.5)
- moved C19 113.0 mm to (44.0, 101.0)
- moved C22 111.4 mm to (60.5, 100.5)
- moved Y2 110.5 mm to (59.5, 97.0), turned to 90 degrees
- moved L10 109.6 mm to (52.0, 95.5)
- moved C17 109.0 mm to (48.0, 95.5)
- moved L11 108.6 mm to (49.5, 91.0), turned to 90 degrees
- moved C11 107.6 mm to (53.5, 93.5)
- moved L13 102.8 mm to (51.0, 81.0), turned to 90 degrees
- moved L21 102.6 mm to (50.5, 93.5)
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- renumbered C5 to C1, C16 to C10, C10 to C11, C7 to C12, C6 to C13, C18 to C14, C19 to C15, C21 to C16, C20 to C17, C17 to C18, C23 to C19, C1 to C2, C9 to C20, C8 to C21, C24 to C22, C25 to C23, C22 to C24, C2 to C3, C11 to C31, C3 to C4, C4 to C5, C12 to C6, C13 to C7, C14 to C8, C15 to C9, L6 to L1, L4 to L10, L3 to L11, L2 to L12, L1 to L13, L7 to L2, L5 to L21, R2 to R1, R1 to R5, U4 to U3, U3 to U4
Connections:
- AE1 pad 2: (no net) -> Earth
- C22 pad 1: Net-(C24-Pad1) -> Net-(Y2-Pad1)
- C23 pad 1: Net-(C25-Pad1) -> Net-(Y2-Pad3)
- IC1 pad 1: unconnected-(IC1-Pad1) -> VDDS
- IC1 pad 12: unconnected-(IC1-Pad12) -> /ADDR
- IC1 pad 13: unconnected-(IC1-Pad13) -> /SDA
- IC1 pad 14: unconnected-(IC1-Pad14) -> /SCL
- IC1 pad 2: unconnected-(IC1-Pad2) -> Earth
- IC1 pad 4: unconnected-(IC1-Pad4) -> Earth
- IC1 pad 5: unconnected-(IC1-Pad5) -> Earth
- IC1 pad 6: unconnected-(IC1-Pad6) -> VDDS
- IC1 pad 7: unconnected-(IC1-Pad7) -> /nCS
- IC1 pad 8: unconnected-(IC1-Pad8) -> /INT1
- IC1 pad 9: unconnected-(IC1-Pad9) -> /INT2
- U4 pad 10: unconnected-(U3-Pad10) -> /DIO_4
- U4 pad 13: unconnected-(U3-Pad13) -> /JTAG_TMSC
- U4 pad 14: unconnected-(U3-Pad14) -> /JTAG_TCKC
- U4 pad 15: unconnected-(U3-Pad15) -> /DIO_5
- U4 pad 16: unconnected-(U3-Pad16) -> /DIO_6
- U4 pad 20: unconnected-(U3-Pad20) -> /DIO_7
- U4 pad 21: unconnected-(U3-Pad21) -> /DIO_8
- U4 pad 22: unconnected-(U3-Pad22) -> /DIO_9
- U4 pad 23: unconnected-(U3-Pad23) -> /DIO_10
- U4 pad 24: unconnected-(U3-Pad24) -> /DIO_11
- U4 pad 25: unconnected-(U3-Pad25) -> /DIO_12
- U4 pad 26: unconnected-(U3-Pad26) -> /DIO_13
- U4 pad 27: unconnected-(U3-Pad27) -> /DIO_14
- U4 pad 30: Net-(U3-Pad30) -> Net-(Y2-Pad1)
- U4 pad 31: Net-(U3-Pad31) -> Net-(Y2-Pad3)
- U4 pad 6: unconnected-(U3-Pad6) -> /DIO_0
- U4 pad 7: unconnected-(U3-Pad7) -> /DIO_1
- U4 pad 8: unconnected-(U3-Pad8) -> /DIO_2
- U4 pad 9: unconnected-(U3-Pad9) -> /DIO_3
- Y2 pad 1: Net-(U3-Pad30) -> Net-(Y2-Pad1)
- Y2 pad 2: Net-(C24-Pad1) -> Earth
- Y2 pad 3: Net-(U3-Pad31) -> Net-(Y2-Pad3)
- Y2 pad 4: Net-(C25-Pad1) -> Earth
Routing:
- net Net-(Y1-Pad1): track 0.00 -> 7.45 mm
- net /RFN: track 0.00 -> 7.40 mm
- net /RX_TX: track 0.00 -> 7.36 mm
- net Net-(C21-Pad2): track 0.00 -> 6.18 mm
- net Net-(Y1-Pad2): track 0.00 -> 5.75 mm
- net /RFP: track 0.00 -> 5.65 mm
- net Net-(L12-Pad2): track 0.00 -> 3.31 mm
- net Net-(L13-Pad2): track 0.00 -> 1.62 mm
- net /DIO_2: track 0.00 -> 1.43 mm, vias 0 -> 1
- net /DIO_1: track 0.00 -> 1.38 mm, vias 0 -> 1
- net /DIO_0: track 0.00 -> 1.05 mm, vias 0 -> 1

Commit message: 2022-06-14 2
Parts:
- moved R4 137.6 mm to (52.5, 61.5), turned to 90 degrees
- moved R3 136.8 mm to (55.0, 44.0), turned to 90 degrees
- moved C8 134.6 mm to (24.0, 46.5)
- moved J2 134.2 mm to (48.8, 62.0), turned to 180 degrees
- moved R2 130.2 mm to (53.0, 44.0), turned to 90 degrees
- moved C16 128.7 mm to (24.0, 51.5), turned to 180 degrees
- moved C15 128.4 mm to (28.5, 54.5), turned to 90 degrees
- moved C10 126.7 mm to (36.5, 49.5), turned to 180 degrees
- moved C14 125.4 mm to (35.0, 45.5), turned to 180 degrees
- moved D1 124.4 mm to (56.5, 61.5), turned to -90 degrees
- moved C7 122.3 mm to (25.0, 57.5), turned to 180 degrees
- moved C9 117.9 mm to (36.5, 48.0), turned to 180 degrees
- moved C24 114.6 mm to (38.0, 52.0), turned to 180 degrees
- moved L1 113.7 mm to (37.0, 55.0), turned to 90 degrees
- moved L2 108.4 mm to (25.0, 54.5), turned to 180 degrees
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Connections:
- J2 pad 1: Earth -> /BATT_STAT
- J2 pad 10: /JTAG_TMSC -> /DIO_9
- J2 pad 11: /DIO_14 -> /DIO_12
- J2 pad 12: /DIO_13 -> /DIO_11
- J2 pad 13: /DIO_12 -> /LED_RED
- J2 pad 14: Earth -> /DIO_13
- J2 pad 15: Earth -> /LED_GREEN
- J2 pad 16: /DIO_11 -> /DIO_14
- J2 pad 17: /DIO_10 -> /SCL
- J2 pad 18: /DIO_9 -> /DIO_0
- J2 pad 19: /DIO_8 -> /SDA
- J2 pad 2: /ADDR -> VDDS
- J2 pad 20: /DIO_7 -> /DIO_1
- J2 pad 21: /DIO_6 -> /ADDR
- J2 pad 22: /DIO_5 -> /DIO_2
- J2 pad 23: /DIO_4 -> /INT2
- J2 pad 25: /DIO_2 -> /INT1
- J2 pad 26: /DIO_1 -> /DIO_4
- J2 pad 27: /DIO_0 -> Earth
- J2 pad 28: VDDS -> Earth
- J2 pad 3: /SCL -> /JTAG_TCKC
- J2 pad 4: /SDA -> /JTAG_TMSC
- J2 pad 5: /INT1 -> /DIO_6
- J2 pad 6: /INT2 -> /DIO_5
- J2 pad 7: /LED_RED -> /DIO_8
- J2 pad 8: /LED_GREEN -> /DIO_7
- J2 pad 9: /JTAG_TCKC -> /DIO_10
Routing:
- net VDDS: track 0.00 -> 95.9 mm, vias 0 -> 4
- net /JTAG_TCKC: track 0.00 -> 30.8 mm, vias 0 -> 1
- net VDDR: track 0.00 -> 30.3 mm, vias 0 -> 3
- net /JTAG_TMSC: track 0.00 -> 29.7 mm, vias 0 -> 1
- net /DIO_4: track 0.00 -> 29.3 mm, vias 0 -> 1
- net /DIO_3: track 0.00 -> 27.2 mm, vias 0 -> 1
- net /DIO_6: track 0.00 -> 26.6 mm, vias 0 -> 1
- net /DIO_5: track 0.00 -> 25.8 mm, vias 0 -> 1
- net /DIO_2: track 1.43 -> 23.3 mm
- net /DIO_8: track 0.00 -> 20.8 mm, vias 0 -> 1
- net /BATT: track 0.00 -> 20.1 mm
- net /DIO_1: track 1.38 -> 21.2 mm
- net /DIO_10: track 0.00 -> 19.6 mm, vias 0 -> 1
- net /DIO_7: track 0.00 -> 18.9 mm, vias 0 -> 1
- net Net-(C1-Pad2): track 0.00 -> 18.9 mm
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- added copper zone on B.Cu, net Earth
- added copper zone on F.Cu, net Earth
Other:
- board outline added: 40 x 55 mm

Commit message: 2022-06-17
Parts:
- added J3: Conn_01x05, Connector_PinHeader_2.54mm:PinHeader_1x05_P2.54mm_Vertical, F.Cu at (22.5, 71.1)
- added J4: Conn_01x10, Connector_PinHeader_2.54mm:PinHeader_1x10_P2.54mm_Vertical, F.Cu at (37.8, 71.1)
- added J5: Conn_01x05, Connector_PinHeader_2.54mm:PinHeader_1x05_P2.54mm_Vertical, F.Cu at (32.7, 48.3)
- added U5: ESP32-C3-MINI-1-N4, ESP32-C4-MINI-1:ESP32-C4-MINI-1, F.Cu at (26.4, 59.7)
- moved C20 20.1 mm to (51.0, 53.5)
- moved R1 20.1 mm to (51.0, 55.5), turned to 0 degrees
- moved J2 20.0 mm to (68.8, 62.0)
- moved AE1 20.0 mm to (51.0, 25.5)
- moved C1 20.0 mm to (67.5, 67.0)
- moved C10 20.0 mm to (56.5, 49.5)
- moved C11 20.0 mm to (53.5, 40.5)
- moved C12 20.0 mm to (50.0, 35.5)
- moved C13 20.0 mm to (51.5, 30.5)
- moved C14 20.0 mm to (55.0, 45.5)
- moved C15 20.0 mm to (48.5, 54.5)
- moved C16 20.0 mm to (44.0, 51.5)
- moved C17 20.0 mm to (48.0, 42.5)
- moved C18 20.0 mm to (44.0, 42.5)
- moved C19 20.0 mm to (44.0, 48.0)
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Routing:
- net Earth: track 13.2 -> 56.8 mm, vias 41 -> 307
- net Net-(U5-Pad23): track 0.00 -> 11.7 mm
- net Net-(U5-Pad12): track 0.00 -> 10.2 mm
- net Net-(U5-Pad22): track 0.00 -> 10.1 mm
- net Net-(U5-Pad13): track 0.00 -> 9.43 mm
- net VDDS: track 95.9 -> 104.8 mm, vias 4 -> 3
- net Net-(U5-Pad21): track 0.00 -> 8.17 mm
- net Net-(U5-Pad20): track 0.00 -> 7.45 mm
- net Net-(U5-Pad16): track 0.00 -> 7.45 mm
- net Net-(U5-Pad18): track 0.00 -> 7.06 mm
- net Net-(U5-Pad31): track 0.00 -> 6.78 mm
- net Net-(U5-Pad19): track 0.00 -> 6.72 mm
- net Net-(U5-Pad8): track 0.00 -> 6.45 mm
- net Net-(U5-Pad3): track 0.00 -> 6.11 mm
- net Net-(U5-Pad30): track 0.00 -> 6.06 mm
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Other:
- board size 40 x 55 mm -> 60 x 55 mm

Commit message: 2022-06-20
Connections:
- AE1 pad 2: Earth -> (no net)
- J2 pad 10: /DIO_9 -> /DIO_5
- J2 pad 11: /DIO_12 -> /DIO_6
- J2 pad 12: /DIO_11 -> /DIO_7
- J2 pad 14: /DIO_13 -> /DIO_8
- J2 pad 16: /DIO_14 -> /DIO_9
- J2 pad 18: /DIO_0 -> /DIO_10
- J2 pad 20: /DIO_1 -> /DIO_11
- J2 pad 22: /DIO_2 -> /DIO_12
- J2 pad 24: /DIO_3 -> /DIO_13
- J2 pad 26: /DIO_4 -> /DIO_14
- J2 pad 3: /JTAG_TCKC -> /DIO_0
- J2 pad 4: /JTAG_TMSC -> /DIO_1
- J2 pad 5: /DIO_6 -> /DIO_2
- J2 pad 6: /DIO_5 -> /DIO_3
- J2 pad 7: /DIO_8 -> /DIO_4
- J2 pad 8: /DIO_7 -> /JTAG_TMSC
- J2 pad 9: /DIO_10 -> /JTAG_TCKC
Routing:
- net /DIO_0: track 19.4 -> 49.9 mm
- net /DIO_1: track 21.2 -> 44.8 mm
- net /DIO_2: track 24.1 -> 44.9 mm
- net Earth: track 56.8 -> 73.9 mm, vias 307 -> 300
- net /DIO_3: track 29.3 -> 38.9 mm
- net /DIO_14: track 16.4 -> 25.6 mm
- net /DIO_13: track 15.3 -> 23.9 mm
- net /DIO_4: track 32.3 -> 39.9 mm
- net /DIO_11: track 15.9 -> 21.3 mm
- net /DIO_12: track 18.2 -> 22.1 mm
- net VDDS: track 104.8 -> 108.4 mm
- net /DIO_9: track 17.1 -> 20.3 mm
- net /DIO_7: track 18.9 -> 20.2 mm
- net /DIO_6: track 26.6 -> 27.2 mm
- net VDDR: track 34.0 -> 33.4 mm
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