File: fishbite.kicad_sch (KiCad schematic)
At the start: 3 parts

Commit message: 2022-06-13
Parts:
- added AE1: Antenna, RF_Antenna:Texas_SWRA117D_2.4GHz_Right, symbol Device:Antenna
- added C1, C2: 4.7uF/2012, Capacitor_SMD:C_0805_2012Metric_Pad1.18x1.45mm_HandSolder, symbol Device:C
- added C10, C6, C8: 1pF/1005, Capacitor_SMD:C_0402_1005Metric_Pad0.74x0.62mm_HandSolder, symbol Device:C
- added C11: 6.8pF/1608, Capacitor_SMD:C_0603_1608Metric_Pad1.08x0.95mm_HandSolder, symbol Device:C
- added C12, C21, C24, C25, C7: DNM, Capacitor_SMD:C_0603_1608Metric_Pad1.08x0.95mm_HandSolder, symbol Device:C
- added C13, C19: 10uF/1608, Capacitor_SMD:C_0603_1608Metric_Pad1.08x0.95mm_HandSolder, symbol Device:C
- added C14, C15, C16, C18, C22, C9: 0.1uF/1608, Capacitor_SMD:C_0603_1608Metric_Pad1.08x0.95mm_HandSolder, symbol Device:C
- added C17, C20: 12pF/1608, Capacitor_SMD:C_0603_1608Metric_Pad1.08x0.95mm_HandSolder, symbol Device:C
- added C23: 1uF/1608, Capacitor_SMD:C_0603_1608Metric_Pad1.08x0.95mm_HandSolder, symbol Device:C
- added C3, C4: 1uF/2012, Capacitor_SMD:C_0805_2012Metric_Pad1.18x1.45mm_HandSolder, symbol Device:C
- added C5: 10uF/3225, Capacitor_SMD:C_1210_3225Metric_Pad1.33x2.70mm_HandSolder, symbol Device:C
- added IC1: ADXL345BCCZ-RL, ADXL345:ADXL345BCCZRL, symbol ADXL345BCCZ-RL:ADXL345BCCZ-RL
- added L1, L2: 2nH, Inductor_SMD:L_0603_1608Metric_Pad1.05x0.95mm_HandSolder, symbol Device:L
- added L3: 2.7nH, Inductor_SMD:L_0603_1608Metric_Pad1.05x0.95mm_HandSolder, symbol Device:L
- added L4: 6.2nH, Inductor_SMD:L_0603_1608Metric_Pad1.05x0.95mm_HandSolder, symbol Device:L
- added L5: 2.4nH, Inductor_SMD:L_0603_1608Metric_Pad1.05x0.95mm_HandSolder, symbol Device:L
- added L6: bead, Inductor_SMD:L_0805_2012Metric_Pad1.05x1.20mm_HandSolder, symbol Device:L_Ferrite
- added L7: 10uH, Inductor_SMD:L_1210_3225Metric_Pad1.42x2.65mm_HandSolder, symbol Device:L
- added R1: 10k/1608, Resistor_SMD:R_0603_1608Metric_Pad0.98x0.95mm_HandSolder, symbol Device:R
- added R2: 100k/1608, Resistor_SMD:R_0603_1608Metric_Pad0.98x0.95mm_HandSolder, symbol Device:R
- added U1: USB4130-GF-C, USB4130:USB4130-GF-C, symbol USB4130:USB4130-GF-C
- added U2: MCP73831-2-OT, Package_TO_SOT_SMD:SOT-23-5, symbol Battery_Management:MCP73831-2-OT
- added Y1: 32.768kHz, Crystal:Crystal_SMD_MicroCrystal_CM9V-T1A-2Pin_1.6x1.0mm_HandSoldering, symbol Device:Crystal
- added Y2: 24MHz, Oscillator:Oscillator_SMD_Abracon_ASE-4Pin_3.2x2.5mm_HandSoldering, symbol Device:Crystal_GND24
- J1: renamed from J?; symbol Connector_Generic:Conn_01x02 -> Connector_Generic_MountingPin:Conn_01x02_MountingPin
- U3: renamed from U?; footprint CC2640R2FRHBR:IC_CC2640R2FRHBR -> Package_DFN_QFN:VQFN-32-1EP_5x5mm_P0.5mm_EP3.1x3.1mm
- gave numbers to parts that had none: 1
Connections:
- net BATT: now reaches U4.1 (VIN)
- net BATT: now also J1.2 (Pin_2), U4.3 (EN), C2.2, C3.2, U2.3 (VBAT)
- net Earth: now reaches U4.2 (GND)
- net Earth: now also J1.1 (Pin_1), J1.MP (MountPin), U3.33 (EGP), C1.1, C10.2, C11.1, C12.1, C13.1, C14.1, C15.1, C16.1, C17.1, C18.1, C19.1, C2.1, C20.2, C21.1, C22.1, C23.1, C24.2, C25.2, C3.1, C4.2, C5.1, C6.1, C7.1, C9.1, R1.2, U1.A12 (GND), U1.B12 (GND), U2.2 (VSS)
- net +3V3: now reaches U4.5 (VOUT)
- net +3V3: now also C4.1, L6.1
- net RFP: now reaches U3.1 (RF_P)
- net RFP: now also C10.1, L4.2
- net VDDS: now reaches U3.11 (VDDS2)
- net VDDS: now also U3.18 (VDDS_DCDC), U3.28 (VDDS), C12.2, C14.2, C16.2, C19.2, C22.2, L6.2, R2.1
- net at U3.12 (DCOUPL): now also C23.2
- net DCDC_SW: now reaches U3.17 (DCDC_SW)
- net DCDC_SW: now also L7.1
- net nRESET: now reaches U3.19 (~{RESET})
- net nRESET: now also C9.2, R2.2
- net RFN: now reaches U3.2 (RF_N)
- net RFN: now also C8.1, L4.1, L5.2
- net VDDR: now reaches U3.29 (VDDR)
- net VDDR: now also U3.32 (VDDR_RF), C13.2, C15.2, C18.2, C21.2, L7.2
- net RX_TX: now reaches U3.3 (RX_TX)
- net RX_TX: now also C11.2, L3.1, L5.1
- net at U3.30 (X24M_N): now also Y2.1
- net at U3.31 (X24M_P): now also Y2.3
- net at U3.4 (X32K_Q1): now also C20.1, Y1.2
- net at U3.5 (X32K_Q2): now also C17.2, Y1.1
- new net: C7.2, C8.2, L2.1, L3.2
- new net: C6.2, L1.1, L2.2
- new net: C1.2, C5.2, U1.A9 (VBUS), U1.B9 (VBUS), U2.4 (VDD)
- new net: R1.1, U2.5 (PROG)
- new net: AE1.1 (A), L1.2
- new net: C24.1, Y2.2
- new net: C25.1, Y2.4
- new net BATT_STAT: U2.1 (STAT)
Other:
- note added: "Pin 11"
- note added: "Pin 18"
- note added: "Pin 28"
- note added: "Pin 29"
- note added: "Pin 32"
- moved on the sheet: U3, U4

Commit message: 2022-06-14
Parts:
- added D1: RG_LED, APBA3010SURKCGKC-GX:APBA3010SURKCGKC-GX, symbol m_LED:LED_Dual_AKK
- added J2: test, Connector_PinHeader_2.54mm:PinHeader_2x14_P2.54mm_Vertical, symbol Connector_Generic:Conn_02x14_Counter_Clockwise
- added R2, R3: 10k/1608, Resistor_SMD:R_0603_1608Metric_Pad0.98x0.95mm_HandSolder, symbol Device:R
- added R4: 100/1608, Resistor_SMD:R_0603_1608Metric_Pad0.98x0.95mm_HandSolder, symbol Device:R
- renumbered C5 to C1, C16 to C10, C10 to C11, C7 to C12, C6 to C13, C18 to C14, C19 to C15, C21 to C16, C20 to C17, C17 to C18, C23 to C19, C1 to C2, C9 to C20, C8 to C21, C24 to C22, C25 to C23, C22 to C24, C2 to C3, C11 to C31, C3 to C4, C4 to C5, C12 to C6, C13 to C7, C14 to C8, C15 to C9, L6 to L1, L4 to L10, L3 to L11, L2 to L12, L1 to L13, L7 to L2, L5 to L21, R2 to R1, R1 to R5, U4 to U3, U3 to U4
Connections:
- net Earth: now also IC1.2 (GND_1), IC1.4 (GND_2), IC1.5 (GND_3), Y2.2, Y2.4, J2.1 (Pin_1), J2.14 (Pin_14), J2.15 (Pin_15)
- net VDDS: now also IC1.1 (VDD_I/O), IC1.6 (VS), J2.28 (Pin_28), R2.1, R3.1, R4.2
- net at U4.30 (X24M_N), Y2.1: now also C22.1
- net at U4.31 (X24M_P), Y2.3: now also C23.1
- net ADDR: now reaches IC1.12 (SDO/ALT_ADDRESS)
- net ADDR: now also J2.2 (Pin_2)
- net SDA: now reaches IC1.13 (SDA/SDI/SDIO)
- net SDA: now also J2.4 (Pin_4), R2.2
- net SCL: now reaches IC1.14 (SCL/SCLK)
- net SCL: now also J2.3 (Pin_3), R3.2
- net nCS: now reaches IC1.7 (~{CS})
- net INT1: now reaches IC1.8 (INT1)
- net INT1: now also J2.5 (Pin_5)
- net INT2: now reaches IC1.9 (INT2)
- net INT2: now also J2.6 (Pin_6)
- net DIO_4: now reaches U4.10 (DIO_4)
- net DIO_4: now also J2.23 (Pin_23)
- net JTAG_TMSC: now reaches U4.13 (JTAG_TMSC)
- net JTAG_TMSC: now also J2.10 (Pin_10)
- net JTAG_TCKC: now reaches U4.14 (JTAG_TCKC)
- net JTAG_TCKC: now also J2.9 (Pin_9)
- net DIO_5: now reaches U4.15 (DIO_5)
- net DIO_5: now also J2.22 (Pin_22)
- net DIO_6: now reaches U4.16 (DIO_6)
- net DIO_6: now also J2.21 (Pin_21)
- net DIO_7: now reaches U4.20 (DIO_7)
- net DIO_7: now also J2.20 (Pin_20)
- net DIO_8: now reaches U4.21 (DIO_8)
- net DIO_8: now also J2.19 (Pin_19)
- net DIO_9: now reaches U4.22 (DIO_9)
- net DIO_9: now also J2.18 (Pin_18)
- net DIO_10: now reaches U4.23 (DIO_10)
- net DIO_10: now also J2.17 (Pin_17)
- net DIO_11: now reaches U4.24 (DIO_11)
- net DIO_11: now also J2.16 (Pin_16)
- net DIO_12: now reaches U4.25 (DIO_12)
- net DIO_12: now also J2.13 (Pin_13)
- net DIO_13: now reaches U4.26 (DIO_13)
- net DIO_13: now also J2.12 (Pin_12)
- net DIO_14: now reaches U4.27 (DIO_14)
- net DIO_14: now also J2.11 (Pin_11)
- net DIO_0: now reaches U4.6 (DIO_0)
- net DIO_0: now also J2.27 (Pin_27)
- net DIO_1: now reaches U4.7 (DIO_1)
- net DIO_1: now also J2.26 (Pin_26)
- net DIO_2: now reaches U4.8 (DIO_2)
- net DIO_2: now also J2.25 (Pin_25)
- net DIO_3: now reaches U4.9 (DIO_3)
- net DIO_3: now also J2.24 (Pin_24)
- new net: D1.1 (A), R4.1
- new net LED_GREEN: D1.3 (K2), J2.8 (Pin_8)
- new net LED_RED: D1.2 (K1), J2.7 (Pin_7)
Other:
- moved on the sheet: IC1

Commit message: 2022-06-14 2
Parts:
- J2: symbol Connector_Generic:Conn_02x14_Counter_Clockwise -> Connector_Generic:Conn_02x14_Odd_Even
Connections:
- net ADDR: now also J2.21 (Pin_21); no longer J2.2 (Pin_2)
- net BATT_STAT: now also J2.1 (Pin_1)
- net DIO_0: now also J2.18 (Pin_18); no longer J2.27 (Pin_27)
- net DIO_1: now also J2.20 (Pin_20); no longer J2.26 (Pin_26)
- net DIO_10: now also J2.9 (Pin_9); no longer J2.17 (Pin_17)
- net DIO_11: now also J2.12 (Pin_12); no longer J2.16 (Pin_16)
- net DIO_12: now also J2.11 (Pin_11); no longer J2.13 (Pin_13)
- net DIO_13: now also J2.14 (Pin_14); no longer J2.12 (Pin_12)
- net DIO_14: now also J2.16 (Pin_16); no longer J2.11 (Pin_11)
- net DIO_2: now also J2.22 (Pin_22); no longer J2.25 (Pin_25)
- net DIO_4: now also J2.26 (Pin_26); no longer J2.23 (Pin_23)
- net DIO_5: now also J2.6 (Pin_6); no longer J2.22 (Pin_22)
- net DIO_6: now also J2.5 (Pin_5); no longer J2.21 (Pin_21)
- net DIO_7: now also J2.8 (Pin_8); no longer J2.20 (Pin_20)
- net DIO_8: now also J2.7 (Pin_7); no longer J2.19 (Pin_19)
- net DIO_9: now also J2.10 (Pin_10); no longer J2.18 (Pin_18)
- net Earth: now also J2.27 (Pin_27), J2.28 (Pin_28); no longer J2.1 (Pin_1), J2.14 (Pin_14), J2.15 (Pin_15)
- net INT1: now also J2.25 (Pin_25); no longer J2.5 (Pin_5)
- net INT2: now also J2.23 (Pin_23); no longer J2.6 (Pin_6)
- net JTAG_TCKC: now also J2.3 (Pin_3); no longer J2.9 (Pin_9)
- net JTAG_TMSC: now also J2.4 (Pin_4); no longer J2.10 (Pin_10)
- net LED_GREEN: now also J2.15 (Pin_15); no longer J2.8 (Pin_8)
- net LED_RED: now also J2.13 (Pin_13); no longer J2.7 (Pin_7)
- net SCL: now also J2.17 (Pin_17); no longer J2.3 (Pin_3)
- net SDA: now also J2.19 (Pin_19); no longer J2.4 (Pin_4)
- net VDDS: now also J2.2 (Pin_2); no longer J2.28 (Pin_28)
Changed lines of the file:
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@@
     (effects (font (size 1.27 1.27)) (justify left bottom))
   )
-  (label "DIO_4" (at 134.62 170.18 0)
+  (label "DIO_4" (at 134.62 187.96 0)
     (effects (font (size 1.27 1.27)) (justify left bottom))
   )
@@
     (effects (font (size 1.27 1.27)) (justify right bottom))
   )
-  (label "DIO_1" (at 134.62 162.56 0)
-    (effects (font (size 1.27 1.27)) (justify left bottom))
-  )
-  (label "JTAG_TMSC" (at 121.92 180.34 180)
-    (effects (font (size 1.27 1.27)) (justify right bottom))
+  (label "DIO_1" (at 134.62 180.34 0)
+    (effects (font (size 1.27 1.27)) (justify left bottom))
+  )
+  (label "JTAG_TMSC" (at 134.62 160.02 0)
+    (effects (font (size 1.27 1.27)) (justify left bottom))
   )
   (label "LED_RED" (at 121.92 172.72 180)
@@
     (effects (font (size 1.27 1.27)) (justify left bottom))
   )
-  (label "DIO_7" (at 134.62 177.8 0)
+  (label "DIO_7" (at 134.62 165.1 0)
     (effects (font (size 1.27 1.27)) (justify left bottom))
   )
@@
     (effects (font (size 1.27 1.27)) (justify left bottom))
   )
-  (label "DIO_12" (at 121.92 187.96 180)
+  (label "DIO_12" (at 121.92 170.18 180)
     (effects (font (size 1.27 1.27)) (justify right bottom))
   )
@@
     (effects (font (size 1.27 1.27)) (justify right bottom))
   )
-  (label "SCL" (at 121.92 162.56 180)
-    (effects (font (size 1.27 1.27)) (justify right bottom))
-  )
-  (label "DIO_2" (at 134.62 165.1 0)
+  (label "SCL" (at 121.92 177.8 180)
+    (effects (font (size 1.27 1.27)) (justify right bottom))
+  )
+  (label "DIO_2" (at 134.62 182.88 0)
     (effects (font (size 1.27 1.27)) (justify left bottom))
   )
@@
     (effects (font (size 1.27 1.27)) (justify left bottom))
   )
-  (label "DIO_14" (at 121.92 182.88 180)
-    (effects (font (size 1.27 1.27)) (justify right bottom))
+  (label "DIO_14" (at 134.62 175.26 0)
+    (effects (font (size 1.27 1.27)) (justify left bottom))
   )
   (label "DIO_0" (at 208.28 97.79 180)
@@
     (effects (font (size 1.27 1.27)) (justify right bottom))
   )
-  (label "DIO_9" (at 134.62 182.88 0)
+  (label "DIO_9" (at 134.62 167.64 0)
     (effects (font (size 1.27 1.27)) (justify left bottom))
   )
@@
     (effects (font (size 1.27 1.27)) (justify left bottom))
   )
-  (label "INT2" (at 121.92 170.18 180)
+  (label "INT2" (at 121.92 185.42 180)
     (effects (font (size 1.27 1.27)) (justify right bottom))
   )
@@
     (effects (font (size 1.27 1.27)) (justify left bottom))
   )
-  (label "DIO_6" (at 134.62 175.26 0)
-    (effects (font (size 1.27 1.27)) (justify left bottom))
+  (label "DIO_6" (at 121.92 162.56 180)
+    (effects (font (size 1.27 1.27)) (justify right bottom))
   )
   (label "INT1" (at 93.98 144.78 0)
@@
     (effects (font (size 1.27 1.27)) (justify left bottom))
   )
-  (label "DIO_3" (at 134.62 167.64 0)
-    (effects (font (size 1.27 1.27)) (justify left bottom))
-  )
-  (label "SDA" (at 121.92 165.1 180)
+  (label "DIO_3" (at 134.62 185.42 0)
+    (effects (font (size 1.27 1.27)) (justify left bottom))
+  )
+  (label "SDA" (at 121.92 180.34 180)
     (effects (font (size 1.27 1.27)) (justify right bottom))
   )
@@
     (effects (font (size 1.27 1.27)) (justify left bottom))
   )
-  (label "ADDR" (at 121.92 160.02 180)
-    (effects (font (size 1.27 1.27)) (justify right bottom))
-  )
-  (label "DIO_5" (at 134.62 172.72 0)
+  (label "ADDR" (at 121.92 182.88 180)
+    (effects (font (size 1.27 1.27)) (justify right bottom))
+  )
+  (label "DIO_5" (at 134.62 162.56 0)
     (effects (font (size 1.27 1.27)) (justify left bottom))
   )
@@
     (effects (font (size 1.27 1.27)) (justify right bottom))
   )
-  (label "JTAG_TCKC" (at 121.92 177.8 180)
-    (effects (font (size 1.27 1.27)) (justify right bottom))
-  )
-  (label "INT1" (at 121.92 167.64 180)
+  (label "JTAG_TCKC" (at 121.92 160.02 180)
+    (effects (font (size 1.27 1.27)) (justify right bottom))
+  )
+  (label "INT1" (at 121.92 187.96 180)
     (effects (font (size 1.27 1.27)) (justify right bottom))
   )
@@
     (effects (font (size 1.27 1.27)) (justify right bottom))
   )
-  (label "DIO_0" (at 134.62 160.02 0)
+  (label "DIO_0" (at 134.62 177.8 0)
     (effects (font (size 1.27 1.27)) (justify left bottom))
   )
@@
     (effects (font (size 1.27 1.27)) (justify left bottom))
   )
-  (label "DIO_11" (at 134.62 187.96 0)
-    (effects (font (size 1.27 1.27)) (justify left bottom))
-  )
-  (label "DIO_8" (at 134.62 180.34 0)
-    (effects (font (size 1.27 1.27)) (justify left bottom))
+  (label "DIO_11" (at 134.62 170.18 0)
+    (effects (font (size 1.27 1.27)) (justify left bottom))
+  )
+  (label "DIO_8" (at 121.92 165.1 180)
+    (effects (font (size 1.27 1.27)) (justify right bottom))
   )
   (label "BATT_STAT" (at 63.5 63.5 90)
     (effects (font (size 1.27 1.27)) (justify left bottom))
   )
-  (label "DIO_10" (at 134.62 185.42 0)
-    (effects (font (size 1.27 1.27)) (justify left bottom))
+  (label "DIO_10" (at 121.92 167.64 180)
+    (effects (font (size 1.27 1.27)) (justify right bottom))
   )
   (label "DIO_10" (at 248.92 105.41 0)
     (effects (font (size 1.27 1.27)) (justify left bottom))
   )
+  (label "BATT_STAT" (at 121.92 157.48 180)
+    (effects (font (size 1.27 1.27)) (justify right bottom))
+  )
   (label "INT2" (at 93.98 142.24 0)
     (effects (font (size 1.27 1.27)) (justify left bottom))
@@
     (effects (font (size 1.27 1.27)) (justify left bottom))
   )
-  (label "DIO_13" (at 121.92 185.42 180)
-    (effects (font (size 1.27 1.27)) (justify right bottom))
+  (label "DIO_13" (at 134.62 172.72 0)
+    (effects (font (size 1.27 1.27)) (justify left bottom))
   )
   (global_label "VDDS" (shape input) (at 201.93 25.4 0) (fields_autoplaced)
@@
     (pin "2")
   )
-  (symbol (lib_id "power:Earth") (at 121.92 157.48 270) (unit 1)
-    (in_bom yes) (on_board yes) (fields_autoplaced)
-    (property "Reference" "#PWR015" (id 0) (at 115.57 157.48 0)
-      (effects (font (size 1.27 1.27)) hide)
-    )
-    (property "Value" "Earth" (id 1) (at 118.11 157.48 0)
-      (effects (font (size 1.27 1.27)) hide)
-    )
-    (property "Footprint" "" (id 2) (at 121.92 157.48 0)
-      (effects (font (size 1.27 1.27)) hide)
-    )
-    (property "Datasheet" "~" (id 3) (at 121.92 157.48 0)
+  (symbol (lib_id "power:Earth") (at 121.92 190.5 270) (unit 1)
+    (in_bom yes) (on_board yes) (fields_autoplaced)
+    (property "Reference" "#PWR015" (id 0) (at 115.57 190.5 0)
+      (effects (font (size 1.27 1.27)) hide)
+    )
+    (property "Value" "Earth" (id 1) (at 118.11 190.5 0)
+      (effects (font (size 1.27 1.27)) hide)
+    )
+    (property "Footprint" "" (id 2) (at 121.92 190.5 0)
+      (effects (font (size 1.27 1.27)) hide)
+    )
+    (property "Datasheet" "~" (id 3) (at 121.92 190.5 0)
       (effects (font (size 1.27 1.27)) hide)
     )
@@
     (pin "1")
   )
-  (symbol (lib_id "Connector_Generic:Conn_02x14_Counter_Clockwise") (at 127 172.72 0) (unit 1)
+  (symbol (lib_id "Connector_Generic:Conn_02x14_Odd_Even") (at 127 172.72 0) (unit 1)
     (in_bom yes) (on_board yes) (fields_autoplaced)
     (property "Reference" "J2" (id 0) (at 128.27 151.13 0))
@@
     (pin "1")
     (pin "2")
-  )
-  (symbol (lib_id "power:Earth") (at 121.92 190.5 270) (unit 1)
-    (in_bom yes) (on_board yes) (fields_autoplaced)
-    (property "Reference" "#PWR016" (id 0) (at 115.57 190.5 0)
-      (effects (font (size 1.27 1.27)) hide)
-    )
-    (property "Value" "Earth" (id 1) (at 118.11 190.5 0)
-      (effects (font (size 1.27 1.27)) hide)
-    )
-    (property "Footprint" "" (id 2) (at 121.92 190.5 0)
-      (effects (font (size 1.27 1.27)) hide)
-    )
-    (property "Datasheet" "~" (id 3) (at 121.92 190.5 0)
-      (effects (font (size 1.27 1.27)) hide)
-    )
-    (pin "1")
   )
   (symbol (lib_id "Device:C") (at 213.36 33.02 180) (unit 1)
@@
       (reference "#PWR015") (unit 1) (value "Earth") (footprint "")
     )
-    (path "/b5e82d3f-8626-4060-a096-a395784a9788"
-      (reference "#PWR016") (unit 1) (value "Earth") (footprint "")
-    )
     (path "/105d2504-17fd-4861-8a71-d7315c4b6623"

Commit message: 2022-06-17
Other:
- added sheet esp32 (esp32.kicad_sch)
Changed lines of the file:
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@@
     (pin "2")
+  )
+  (sheet (at 125.73 46.99) (size 16.51 12.7) (fields_autoplaced)
+    (stroke (width 0.1524) (type solid) (color 0 0 0 0))
+    (fill (color 0 0 0 0.0000))
+    (property "Sheet name" "esp32" (id 0) (at 125.73 46.2784 0)
+      (effects (font (size 1.27 1.27)) (justify left bottom))
+    )
+    (property "Sheet file" "esp32.kicad_sch" (id 1) (at 125.73 60.2746 0)
+      (effects (font (size 1.27 1.27)) (justify left top))
+    )
   )
   (sheet_instances
     (path "/" (page "1"))
+    (path "/f7aa75c5-0bfb-4814-b8eb-5f8a9a128aa9" (page "2"))
   )
   (symbol_instances
@@
       (reference "#PWR038") (unit 1) (value "Earth") (footprint "")
     )
+    (path "/f7aa75c5-0bfb-4814-b8eb-5f8a9a128aa9/26ba45e2-e91d-4dba-bb41-b1e0c5d3e276"
+      (reference "#PWR0101") (unit 1) (value "Earth") (footprint "")
+    )
+    (path "/f7aa75c5-0bfb-4814-b8eb-5f8a9a128aa9/bbe5c00c-19fc-4d57-bdaf-434080a9cd15"
+      (reference "#PWR0102") (unit 1) (value "Earth") (footprint "")
+    )
+    (path "/f7aa75c5-0bfb-4814-b8eb-5f8a9a128aa9/00cbc649-24f1-4303-ba33-cd561c64548c"
+      (reference "#PWR0103") (unit 1) (value "Earth") (footprint "")
+    )
     (path "/a4ff6661-b15b-4171-85d2-7974fa9df9ae"
       (reference "AE1") (unit 1) (value "Antenna") (footprint "RF_Antenna:Texas_SWRA117D_2.4GHz_Right")
@@
       (reference "J2") (unit 1) (value "test") (footprint "Connector_PinHeader_2.54mm:PinHeader_2x14_P2.54mm_Vertical")
     )
+    (path "/f7aa75c5-0bfb-4814-b8eb-5f8a9a128aa9/493c8b2b-f59a-4b8b-8bcf-44e4a2d8e4a2"
+      (reference "J3") (unit 1) (value "Conn_01x05") (footprint "Connector_PinHeader_2.54mm:PinHeader_1x05_P2.54mm_Vertical")
+    )
+    (path "/f7aa75c5-0bfb-4814-b8eb-5f8a9a128aa9/3eae3ba7-df0f-47b3-8c65-92aa25035e52"
+      (reference "J4") (unit 1) (value "Conn_01x10") (footprint "Connector_PinHeader_2.54mm:PinHeader_1x10_P2.54mm_Vertical")
+    )
+    (path "/f7aa75c5-0bfb-4814-b8eb-5f8a9a128aa9/ae10f519-4b80-4b5e-b6f6-f46c02d44d99"
+      (reference "J5") (unit 1) (value "Conn_01x05") (footprint "Connector_PinHeader_2.54mm:PinHeader_1x05_P2.54mm_Vertical")
+    )
     (path "/306d0f60-f326-49e0-aea4-c110dff4ff31"
       (reference "L1") (unit 1) (value "bead") (footprint "Inductor_SMD:L_0805_2012Metric_Pad1.05x1.20mm_HandSolder")
@@
       (reference "U4") (unit 1) (value "CC2640R2FRHBR") (footprint "Package_DFN_QFN:VQFN-32-1EP_5x5mm_P0.5mm_EP3.1x3.1mm")
     )
+    (path "/f7aa75c5-0bfb-4814-b8eb-5f8a9a128aa9/21b4a2e6-0e40-4192-943e-bb939e580e2b"
+      (reference "U5") (unit 1) (value "ESP32-C3-MINI-1-N4") (footprint "ESP32-C4-MINI-1:ESP32-C4-MINI-1")
+    )
     (path "/d931cd6a-223e-4c0b-bfcf-8fae9ceabb74"
