File: fishbite.kicad_sch (KiCad schematic)
At the start: 48 parts, among them IC1 ADXL345BCCZ-RL, J1 Batt, J2 test, U1 USB4130-GF-C, U2 MCP73831-2-OT, U3 MIC5317-3.3YM5-TR, U4 CC2640R2FRHBR, Y1 32.768kHz, Y2 24MHz

Commit message: 2022-06-20
Connections:
- net DIO_0: now also J2.3 (Pin_3); no longer J2.18 (Pin_18)
- net DIO_1: now also J2.4 (Pin_4); no longer J2.20 (Pin_20)
- net DIO_10: now also J2.18 (Pin_18); no longer J2.9 (Pin_9)
- net DIO_11: now also J2.20 (Pin_20); no longer J2.12 (Pin_12)
- net DIO_12: now also J2.22 (Pin_22); no longer J2.11 (Pin_11)
- net DIO_13: now also J2.24 (Pin_24); no longer J2.14 (Pin_14)
- net DIO_14: now also J2.26 (Pin_26); no longer J2.16 (Pin_16)
- net DIO_2: now also J2.5 (Pin_5); no longer J2.22 (Pin_22)
- net DIO_3: now also J2.6 (Pin_6); no longer J2.24 (Pin_24)
- net DIO_4: now also J2.7 (Pin_7); no longer J2.26 (Pin_26)
- net DIO_5: now also J2.10 (Pin_10); no longer J2.6 (Pin_6)
- net DIO_6: now also J2.11 (Pin_11); no longer J2.5 (Pin_5)
- net DIO_7: now also J2.12 (Pin_12); no longer J2.8 (Pin_8)
- net DIO_8: now also J2.14 (Pin_14); no longer J2.7 (Pin_7)
- net DIO_9: now also J2.16 (Pin_16); no longer J2.10 (Pin_10)
- net JTAG_TCKC: now also J2.9 (Pin_9); no longer J2.3 (Pin_3)
- net JTAG_TMSC: now also J2.8 (Pin_8); no longer J2.4 (Pin_4)
Changed lines of the file:
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@@
     (effects (font (size 1.27 1.27)) (justify left bottom))
   )
-  (label "DIO_4" (at 134.62 187.96 0)
-    (effects (font (size 1.27 1.27)) (justify left bottom))
+  (label "DIO_4" (at 121.92 165.1 180)
+    (effects (font (size 1.27 1.27)) (justify right bottom))
   )
   (label "DIO_6" (at 208.28 113.03 180)
@@
     (effects (font (size 1.27 1.27)) (justify right bottom))
   )
-  (label "DIO_1" (at 134.62 180.34 0)
+  (label "DIO_1" (at 134.62 160.02 0)
     (effects (font (size 1.27 1.27)) (justify left bottom))
   )
-  (label "JTAG_TMSC" (at 134.62 160.02 0)
+  (label "JTAG_TMSC" (at 134.62 165.1 0)
     (effects (font (size 1.27 1.27)) (justify left bottom))
   )
@@
     (effects (font (size 1.27 1.27)) (justify left bottom))
   )
-  (label "DIO_7" (at 134.62 165.1 0)
+  (label "DIO_7" (at 134.62 170.18 0)
     (effects (font (size 1.27 1.27)) (justify left bottom))
   )
@@
     (effects (font (size 1.27 1.27)) (justify left bottom))
   )
-  (label "DIO_12" (at 121.92 170.18 180)
-    (effects (font (size 1.27 1.27)) (justify right bottom))
+  (label "DIO_12" (at 134.62 182.88 0)
+    (effects (font (size 1.27 1.27)) (justify left bottom))
   )
   (label "DIO_8" (at 248.92 100.33 0)
@@
     (effects (font (size 1.27 1.27)) (justify right bottom))
   )
-  (label "DIO_2" (at 134.62 182.88 0)
-    (effects (font (size 1.27 1.27)) (justify left bottom))
+  (label "DIO_2" (at 121.92 162.56 180)
+    (effects (font (size 1.27 1.27)) (justify right bottom))
   )
   (label "DIO_9" (at 248.92 102.87 0)
@@
     (effects (font (size 1.27 1.27)) (justify left bottom))
   )
-  (label "DIO_14" (at 134.62 175.26 0)
+  (label "DIO_14" (at 134.62 187.96 0)
     (effects (font (size 1.27 1.27)) (justify left bottom))
   )
@@
     (effects (font (size 1.27 1.27)) (justify right bottom))
   )
-  (label "DIO_9" (at 134.62 167.64 0)
+  (label "DIO_9" (at 134.62 175.26 0)
     (effects (font (size 1.27 1.27)) (justify left bottom))
   )
@@
     (effects (font (size 1.27 1.27)) (justify left bottom))
   )
-  (label "DIO_6" (at 121.92 162.56 180)
+  (label "DIO_6" (at 121.92 170.18 180)
     (effects (font (size 1.27 1.27)) (justify right bottom))
   )
@@
     (effects (font (size 1.27 1.27)) (justify left bottom))
   )
-  (label "DIO_3" (at 134.62 185.42 0)
+  (label "DIO_3" (at 134.62 162.56 0)
     (effects (font (size 1.27 1.27)) (justify left bottom))
   )
@@
     (effects (font (size 1.27 1.27)) (justify right bottom))
   )
-  (label "DIO_5" (at 134.62 162.56 0)
+  (label "DIO_5" (at 134.62 167.64 0)
     (effects (font (size 1.27 1.27)) (justify left bottom))
   )
@@
     (effects (font (size 1.27 1.27)) (justify right bottom))
   )
-  (label "JTAG_TCKC" (at 121.92 160.02 180)
+  (label "JTAG_TCKC" (at 121.92 167.64 180)
     (effects (font (size 1.27 1.27)) (justify right bottom))
   )
@@
     (effects (font (size 1.27 1.27)) (justify right bottom))
   )
-  (label "DIO_0" (at 134.62 177.8 0)
-    (effects (font (size 1.27 1.27)) (justify left bottom))
+  (label "DIO_0" (at 121.92 160.02 180)
+    (effects (font (size 1.27 1.27)) (justify right bottom))
   )
   (label "DIO_13" (at 248.92 113.03 0)
     (effects (font (size 1.27 1.27)) (justify left bottom))
   )
-  (label "DIO_11" (at 134.62 170.18 0)
+  (label "DIO_11" (at 134.62 180.34 0)
     (effects (font (size 1.27 1.27)) (justify left bottom))
   )
-  (label "DIO_8" (at 121.92 165.1 180)
-    (effects (font (size 1.27 1.27)) (justify right bottom))
+  (label "DIO_8" (at 134.62 172.72 0)
+    (effects (font (size 1.27 1.27)) (justify left bottom))
   )
   (label "BATT_STAT" (at 63.5 63.5 90)
     (effects (font (size 1.27 1.27)) (justify left bottom))
   )
-  (label "DIO_10" (at 121.92 167.64 180)
-    (effects (font (size 1.27 1.27)) (justify right bottom))
+  (label "DIO_10" (at 134.62 177.8 0)
+    (effects (font (size 1.27 1.27)) (justify left bottom))
   )
   (label "DIO_10" (at 248.92 105.41 0)
@@
     (effects (font (size 1.27 1.27)) (justify left bottom))
   )
-  (label "DIO_13" (at 134.62 172.72 0)
+  (label "DIO_13" (at 134.62 185.42 0)
     (effects (font (size 1.27 1.27)) (justify left bottom))
   )
